Commit message: Fix bugs in origin urdf

File: description/urdf/yahboomcar_R2.urdf.xacro (robot description, xacro)
@@ -5,5 +5,11 @@
 <robot name="yahboomcar_R2" xmlns:xacro="http://ros.org/wiki/xacro">
   <!--xacro:include filename="$(find description)/urdf/yahboomcar_R2.gazebo.xacro"/-->
-  <link name="imu_link"/>
+  <link name="base_footprint">
+  </link>
+  <joint name="base_joint" type="fixed">
+    <parent link="base_footprint"/>
+    <child link="base_link"/>
+    <origin xyz="0.0 0.0 0.0215" rpy="0 0 0"/>
+  </joint>
   <link name="base_link">
     <inertial>
@@ -248,5 +254,5 @@
       link="front_left_wheel" />
     <axis
-      xyz="0 -1 0" />
+      xyz="0 1 0" />
   </joint>
   <link name="front_right_steer">
@@ -406,5 +412,5 @@
   </joint>
   <link name="laser_link">
-    <inertial>
+    <!-- <inertial>
       <origin
         xyz="0 0 0"
@@ -419,5 +425,5 @@
         iyz="0"
         izz="0" />
-    </inertial>
+    </inertial> -->
     <visual>
       <origin
@@ -455,4 +461,6 @@
       xyz="0 0 0" />
   </joint>
+  <link name="imu_link">
+  </link>
   <joint name="base_imu" type="fixed">
     <parent link="base_link"/>
@@ -460,11 +468,6 @@
     <origin xyz="-0.05 0.0 0.05" rpy="0 3.1415 1.5707"/>
   </joint>
-  <link name="base_footprint"/>
-  <joint name="base_joint" type="fixed">
-    <parent link="base_footprint"/>
-    <child link="base_link"/>
-    <origin xyz="0.0 0.0 0.0215" rpy="0 0 0"/>
-  </joint>
-  <!--<transmission name="front_right_steer_joint_trans">
+  <!--
+  <transmission name="front_right_steer_joint_trans">
     <type>transmission_interface/SimpleTransmission</type>
     <joint name="front_right_steer_joint" >
@@ -507,4 +510,5 @@
       <mechanicalReduction>1</mechanicalReduction>
     </actuator>
-  </transmission>-->
+  </transmission>
+  -->
 </robot>
