Commit message: Port ackermann ros2_control & gazebo_control FIXME: front wheel slips when linear.x speed > 2 under ros2_control

File: description/urdf/prius.urdf.xacro (robot description, xacro)
@@ -1,994 +1,12 @@
 <?xml version="1.0"?>
-<robot xmlns:xacro="http://ros.org/wiki/xacro" name="prius">
-  <!--- Surface properties must come first? -->
-  <gazebo reference="front_left_wheel">
-    <mu1>0.9</mu1>
-    <mu2>0.9</mu2>
-    <minDepth>0.005</minDepth>
-    <kp>1e8</kp>
-  </gazebo>
-  <gazebo reference="front_right_wheel">
-    <mu1>0.9</mu1>
-    <mu2>0.9</mu2>
-    <minDepth>0.005</minDepth>
-    <kp>1e8</kp>
-  </gazebo>
-  <gazebo reference="rear_left_wheel">
-    <mu1>0.9</mu1>
-    <mu2>0.9</mu2>
-    <minDepth>0.005</minDepth>
-    <kp>1e8</kp>
-  </gazebo>
-  <gazebo reference="rear_right_wheel">
-    <mu1>0.9</mu1>
-    <mu2>0.9</mu2>
-    <minDepth>0.005</minDepth>
-    <kp>1e8</kp>
-  </gazebo>
-  <link name="base_link">
-    <inertial>
-      <mass value="1"/>
-      <inertia ixx="0.001" ixy="0.0" ixz="0.0" iyy="0.001" iyz="0.0" izz="0.001"/>
-    </inertial>
-  </link>
-  <joint name="base_link_connection" type="fixed">
-    <parent link="base_link"/>
-    <child link="chassis"/>
-    <origin xyz="1.45 0 0" rpy="0 0 1.57"/>
-    <axis xyz="1 0 0"/>
-  </joint>
-  <link name="chassis">
-    <visual>
-      <origin xyz="0 0 0" rpy="0 0 0"/>
-      <geometry>
-        <mesh filename="package://description/meshes/hybrid_body.obj" scale="0.01 0.01 0.01"/>
-      </geometry>
-    </visual>
-    <collision name="chassis">
-      <origin xyz="0.0 0.05 0.625" rpy="0 0 0"/>
-      <geometry>
-        <box size="1.7526 2.1 0.95"/>
-      </geometry>
-    </collision>
-    <collision name="front_bumper">
-      <origin xyz="0.0 -2.0 0.458488" rpy="0.0 0 0"/>
-      <geometry>
-        <box size="1.337282 0.48 0.566691"/>
-      </geometry>
-    </collision>
-    <collision name="hood">
-      <origin xyz="0.0 -1.900842 0.676305" rpy="0.341247 0 0"/>
-      <geometry>
-        <box size="1.597968 0.493107 0.265468"/>
-      </geometry>
-    </collision>
-    <collision name="windshield">
-      <origin xyz="0.0 -0.875105 1.032268" rpy="0.335476 0 0"/>
-      <geometry>
-        <box size="1.168381 1.654253 0.272347"/>
-      </geometry>
-    </collision>
-    <collision name="top_front">
-      <origin xyz="0.0 0.161236 1.386042" rpy="0.135030 0 0"/>
-      <geometry>
-        <box size="1.279154 0.625988 0.171868"/>
-      </geometry>
-    </collision>
-    <collision name="top_rear">
-      <origin xyz="0.0 0.817696 1.360069" rpy="-0.068997 0 0"/>
-      <geometry>
-        <box size="1.285130 0.771189 0.226557"/>
-      </geometry>
-    </collision>
-    <collision name="rear_window">
-      <origin xyz="0.0 1.640531 1.175126" rpy="-0.262017 0 0"/>
-      <geometry>
-        <box size="1.267845 1.116344 0.244286"/>
-      </geometry>
-    </collision>
-    <collision name="trunk">
-      <origin xyz="0.0 1.637059 0.888180" rpy="0.0 0 0"/>
-      <geometry>
-        <box size="1.788064 1.138988 0.482746"/>
-      </geometry>
-    </collision>
-    <collision name="back_bumper">
-      <origin xyz="0.0 2.054454 0.577870" rpy="0.0 0 0"/>
-      <geometry>
-        <box size="1.781650 0.512093 0.581427"/>
-      </geometry>
-    </collision>
-    <inertial>
-      <mass value="1356.0"/>
-      <origin xyz="0 0 0.48" rpy="0 0 1.5708"/>
-      <inertia ixx="2581.13354740" ixy="0.0" ixz="0.0" iyy="591.30846112" iyz="0.0" izz="2681.95008628"/>
-    </inertial>
-  </link>
-  <link name="fl_axle">
-    <inertial>
-      <mass value="1"/>
-      <origin xyz="0 0 0"/>
-      <inertia ixx="0.004" ixy="0.0" ixz="0.0" iyy="0.004" iyz="0.0" izz="0.004"/>
-    </inertial>
-  </link>
-  <link name="fr_axle">
-    <inertial>
-      <mass value="1"/>
-      <origin xyz="0 0 0"/>
-      <inertia ixx="0.004" ixy="0.0" ixz="0.0" iyy="0.004" iyz="0.0" izz="0.004"/>
-    </inertial>
-  </link>
-  <link name="front_left_wheel">
-    <inertial>
-      <mass value="11"/>
-      <origin xyz="0 0 0"/>
-      <inertia ixx="0.58631238" ixy="0.0" ixz="0.0" iyy="0.33552910" iyz="0.0" izz="0.33552910"/>
-    </inertial>
-    <collision name="front_left_wheel_collision">
-      <geometry>
-        <sphere radius="0.31265"/>
-      </geometry>
-    </collision>
-    <visual>
-      <origin xyz="0 0 0" rpy="0 0 0"/>
-      <geometry>
-        <mesh filename="package://description/meshes/wheel.obj" scale="0.01 0.01 0.01"/>
-      </geometry>
-    </visual>
-  </link>
-  <link name="front_right_wheel">
-    <inertial>
-      <mass value="11"/>
-      <origin xyz="0 0 0"/>
-      <inertia ixx="0.58631238" ixy="0.0" ixz="0.0" iyy="0.33552910" iyz="0.0" izz="0.33552910"/>
-    </inertial>
-    <collision name="front_right_wheel_collision">
-      <geometry>
-        <sphere radius="0.31265"/>
-      </geometry>
-    </collision>
-    <visual>
-      <origin xyz="0 0 0" rpy="0 0 0"/>
-      <geometry>
-        <mesh filename="package://description/meshes/wheel.obj" scale="0.01 0.01 0.01"/>
-      </geometry>
-    </visual>
-  </link>
-  <link name="rear_left_wheel">
-    <inertial>
-      <mass value="11"/>
-      <origin xyz="0 0 0"/>
-      <inertia ixx="0.58631238" ixy="0.0" ixz="0.0" iyy="0.33552910" iyz="0.0" izz="0.33552910"/>
-    </inertial>
-    <collision name="rear_left_wheel_collision">
-      <geometry>
-        <sphere radius="0.31265"/>
-      </geometry>
-    </collision>
-    <visual>
-      <origin xyz="0 0 0" rpy="0 0 0"/>
-      <geometry>
-        <mesh filename="package://description/meshes/wheel.obj" scale="0.01 0.01 0.01"/>
-      </geometry>
-    </visual>
-  </link>
-  <link name="rear_right_wheel">
-    <inertial>
-      <mass value="11"/>
-      <origin xyz="0 0 0"/>
-      <inertia ixx="0.58631238" ixy="0.0" ixz="0.0" iyy="0.33552910" iyz="0.0" izz="0.33552910"/>
-    </inertial>
-    <collision name="rear_right_wheel_collision">
-      <geometry>
-        <sphere radius="0.31265"/>
-      </geometry>
-    </collision>
-    <visual>
-      <origin xyz="0 0 0" rpy="0 0 0"/>
-      <geometry>
-        <mesh filename="package://description/meshes/wheel.obj" scale="0.01 0.01 0.01"/>
-      </geometry>
-    </visual>
-  </link>
-  <link name="steering_wheel">
-    <inertial>
-      <mass value="1.0"/>
-      <inertia ixx="0.14583300" ixy="0.0" ixz="0.0" iyy="0.14583300" iyz="0.0" izz="0.125"/>
-    </inertial>
-    <visual>
-      <origin xyz="0 0 0" rpy="1.302101 0 0"/>
-      <geometry>
-        <mesh filename="package://description/meshes/steering_wheel.obj" scale="0.01 0.01 0.01"/>
-      </geometry>
-    </visual>
-  </link>
-  <joint name="steering_joint" type="continuous">
-    <origin xyz="0.357734 -0.627868 0.988243" rpy="-1.302101 0 0"/>
-    <parent link="chassis"/>
-    <child link="steering_wheel"/>
-    <axis xyz="0 0 1"/>
-    <limit lower="-7.85" upper="7.85" effort="10000000" velocity="1000000"/>
-  </joint>
-  <joint name="front_left_steer_joint" type="continuous">
-    <parent link="chassis"/>
-    <child link="fl_axle"/>
-    <origin xyz="0.767 -1.41 0.3" rpy="0 0 0"/>
-    <axis xyz="0 0 1"/>
-    <limit lower="-0.8727" upper="0.8727" effort="10000000" velocity="1000000"/>
-  </joint>
-  <joint name="front_right_steer_joint" type="continuous">
-    <parent link="chassis"/>
-    <child link="fr_axle"/>
-    <origin xyz="-0.767 -1.41 0.3" rpy="0 0 0"/>
-    <axis xyz="0 0 1"/>
-    <limit lower="-0.8727" upper="0.8727" effort="10000000" velocity="1000000"/>
-  </joint>
-  <joint name="front_left_wheel_joint" type="continuous">
-    <parent link="fl_axle"/>
-    <child link="front_left_wheel"/>
-    <origin xyz="0 0 0" rpy="0 0 0"/>
-    <axis xyz="1 0 0"/>
-  </joint>
-  <joint name="front_right_wheel_joint" type="continuous">
-    <parent link="fr_axle"/>
-    <child link="front_right_wheel"/>
-    <origin xyz="0 0 0" rpy="0 0 0"/>
-    <axis xyz="1 0 0"/>
-  </joint>
-  <joint name="rear_left_wheel_joint" type="continuous">
-    <parent link="chassis"/>
-    <child link="rear_left_wheel"/>
-    <origin xyz="0.793 1.45 0.3" rpy="0 0 0"/>
-    <axis xyz="1 0 0"/>
-  </joint>
-  <joint name="rear_right_wheel_joint" type="continuous">
-    <parent link="chassis"/>
-    <child link="rear_right_wheel"/>
-    <origin xyz="-0.793 1.45 0.3" rpy="0 0 0"/>
-    <axis xyz="1 0 0"/>
-  </joint>
-  <!-- Sensor links and fixed joints -->
-  <link name="center_laser_link">
-    <inertial>
-      <mass value="1"/>
-      <inertia ixx="0.001" ixy="0.0" ixz="0.0" iyy="0.001" iyz="0.0" izz="0.001"/>
-    </inertial>
-  </link>
-  <joint name="center_laser_joint" type="fixed">
-    <parent link="chassis"/>
-    <child link="center_laser_link"/>
-    <origin xyz="0 0.4 1.8" rpy="0 0 -1.5707"/>
-  </joint>
-  <link name="front_left_laser_link">
-    <inertial>
-      <mass value="1"/>
-      <inertia ixx="0.001" ixy="0.0" ixz="0.0" iyy="0.001" iyz="0.0" izz="0.001"/>
-    </inertial>
-  </link>
-  <joint name="front_left_laser_joint" type="fixed">
-    <parent link="chassis"/>
-    <child link="front_left_laser_link"/>
-    <origin xyz="1 -2.3 0.5" rpy="0 0.05 0"/>
-  </joint>
-  <link name="front_right_laser_link">
-    <inertial>
-      <mass value="1"/>
-      <inertia ixx="0.001" ixy="0.0" ixz="0.0" iyy="0.001" iyz="0.0" izz="0.001"/>
-    </inertial>
-  </link>
-  <joint name="front_right_laser_joint" type="fixed">
-    <parent link="chassis"/>
-    <child link="front_right_laser_link"/>
-    <origin xyz="-1 -2.3 0.5" rpy="0 0.05 3.14"/>
-  </joint>
-  <gazebo reference="base_link_connection">
-    <disableFixedJointLumping>true</disableFixedJointLumping>
-  </gazebo>
-  <link name="front_camera_link">
-    <inertial>
-      <mass value="1"/>
-      <inertia ixx="0.001" ixy="0.0" ixz="0.0" iyy="0.001" iyz="0.0" izz="0.001"/>
-    </inertial>
-  </link>
-  <joint name="front_camera_joint" type="fixed">
-    <parent link="chassis"/>
-    <child link="front_camera_link"/>
-    <origin xyz="0 -0.4 1.4" rpy="0 0.05 -1.5707"/>
-  </joint>
-  <link name="front_camera_link_optical">
-    <inertial>
-      <mass value="1"/>
-      <inertia ixx="0.001" ixy="0.0" ixz="0.0" iyy="0.001" iyz="0.0" izz="0.001"/>
-    </inertial>
-  </link>
-  <joint name="front_camera_optical_joint" type="fixed">
-    <origin xyz="0 0 0" rpy="-1.5707 0 -1.5707"/>
-    <parent link="front_camera_link"/>
-    <child link="front_camera_link_optical"/>
-  </joint>
-  <link name="back_camera_link">
-    <inertial>
-      <mass value="1"/>
-      <inertia ixx="0.001" ixy="0.0" ixz="0.0" iyy="0.001" iyz="0.0" izz="0.001"/>
-    </inertial>
-  </link>
-  <joint name="back_camera_joint" type="fixed">
-    <parent link="chassis"/>
-    <child link="back_camera_link"/>
-    <origin xyz="0 1.45 1.4" rpy="0 0.05 1.5707"/>
-  </joint>
-  <link name="back_camera_link_optical">
-    <inertial>
-      <mass value="1"/>
-      <inertia ixx="0.001" ixy="0.0" ixz="0.0" iyy="0.001" iyz="0.0" izz="0.001"/>
-    </inertial>
-  </link>
-  <joint name="back_camera_optical_joint" type="fixed">
-    <origin xyz="0 0 0" rpy="-1.5707 0 -1.5707"/>
-    <parent link="back_camera_link"/>
-    <child link="back_camera_link_optical"/>
-  </joint>
-  <link name="left_camera_link">
-    <inertial>
-      <mass value="1"/>
-      <inertia ixx="0.001" ixy="0.0" ixz="0.0" iyy="0.001" iyz="0.0" izz="0.001"/>
-    </inertial>
-  </link>
-  <joint name="left_camera_joint" type="fixed">
-    <parent link="chassis"/>
-    <child link="left_camera_link"/>
-    <origin xyz="1 -0.7 1.0" rpy="0 0.05 1.0"/>
-  </joint>
-  <link name="left_camera_link_optical">
-    <inertial>
-      <mass value="1"/>
-      <inertia ixx="0.001" ixy="0.0" ixz="0.0" iyy="0.001" iyz="0.0" izz="0.001"/>
-    </inertial>
-  </link>
-  <joint name="left_camera_optical_joint" type="fixed">
-    <origin xyz="0 0 0" rpy="-1.5707 0 -1.5707"/>
-    <parent link="left_camera_link"/>
-    <child link="left_camera_link_optical"/>
-  </joint>
-  <link name="right_camera_link">
-    <inertial>
-      <mass value="1"/>
-      <inertia ixx="0.001" ixy="0.0" ixz="0.0" iyy="0.001" iyz="0.0" izz="0.001"/>
-    </inertial>
-  </link>
-  <joint name="right_camera_joint" type="fixed">
-    <parent link="chassis"/>
-    <child link="right_camera_link"/>
-    <origin xyz="-1 -0.7 1.0" rpy="0 0.05 2.1416"/>
-  </joint>
-  <link name="right_camera_link_optical">
-    <inertial>
-      <mass value="1"/>
-      <inertia ixx="0.001" ixy="0.0" ixz="0.0" iyy="0.001" iyz="0.0" izz="0.001"/>
-    </inertial>
-  </link>
-  <joint name="right_camera_optical_joint" type="fixed">
-    <origin xyz="0 0 0" rpy="-1.5707 0 -1.5707"/>
-    <parent link="right_camera_link"/>
-    <child link="right_camera_link_optical"/>
-  </joint>
-  <link name="back_left_far_sonar_link">
-    <inertial>
-      <mass value="1"/>
-      <inertia ixx="0.001" ixy="0.0" ixz="0.0" iyy="0.001" iyz="0.0" izz="0.001"/>
-    </inertial>
-  </link>
-  <joint name="back_left_far_sonar_joint" type="fixed">
-    <parent link="chassis"/>
-    <child link="back_left_far_sonar_link"/>
-    <origin xyz="0.7 2.4 0.5" rpy="0 0 1.5707"/>
-  </joint>
-  <link name="back_left_middle_sonar_link">
-    <inertial>
-      <mass value="1"/>
-      <inertia ixx="0.001" ixy="0.0" ixz="0.0" iyy="0.001" iyz="0.0" izz="0.001"/>
-    </inertial>
-  </link>
-  <joint name="back_left_middle_sonar_joint" type="fixed">
-    <parent link="chassis"/>
-    <child link="back_left_middle_sonar_link"/>
-    <origin xyz="0.24 2.4 0.5" rpy="0 0 1.5707"/>
-  </joint>
-  <link name="back_right_far_sonar_link">
-    <inertial>
-      <mass value="1"/>
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