Commit message: Fix decimal point typo, but problem still not solved

File: description/urdf/autocar_core.xacro (robot description, xacro)
@@ -174,5 +174,5 @@
     </inertial>
   </link>
-  <link name="steering_wheel" />
+  <link name="steering_wheel" />  <!-- FIXME: missing inertia, error in rviz2 -->
   <joint name="br_axle" type="continuous">
     <origin rpy="0 0 0" xyz="0.8750 -1.013637 -0.144363" />

File: description/urdf/autocar_gazebo_control.xacro (robot description, xacro)
@@ -19,5 +19,5 @@
       <!-- Max absolute steer angle for tyre in radians-->
       <!-- Any cmd_vel angular z greater than this would be capped -->
-      <max_steer>0,85</max_steer>
+      <max_steer>0.85</max_steer>
       <!-- Max absolute steering angle of steering wheel -->
       <max_steering_angle>7.85</max_steering_angle>

Commit message: Fix commit c8c6934 by changing collision of rear wheels from mesh file to cylinder of geometry mentioned in the original author's model.sdf file. NOTE: But still don't know why the mesh file collision won't work?

File: description/urdf/autocar_core.xacro (robot description, xacro)
@@ -94,8 +94,14 @@
     </visual>
     <collision>
+      <!-- NOTE: Somehow libgazebo_ros_ackermann_drive.so don't work with collision using this custom mesh. Only built-in cylinder and sphere works, and built-in box don't work either.
       <origin rpy="0 0 0" xyz="-0.8750 1.0136 0.1444" />
       <geometry>
         <mesh filename="file://$(find description)/meshes/br_1.stl" scale="0.001 0.001 0.001" />
       </geometry>
+      -->
+      <origin xyz="0 0 0" rpy="0 1.5708 0"/>
+      <geometry>
+        <cylinder radius="0.3425" length="0.22"/>
+      </geometry>
     </collision>
   </link>
@@ -114,7 +120,13 @@
     </visual>
     <collision>
+      <!-- NOTE: Somehow libgazebo_ros_ackermann_drive.so don't work with collision using this custom mesh. Only built-in cylinder and sphere works, and built-in box don't work either.
       <origin rpy="0 0 0" xyz="0.8750 1.0136 0.1444" />
       <geometry>
         <mesh filename="file://$(find description)/meshes/bl_1.stl" scale="0.001 0.001 0.001" />
+      </geometry>
+      -->
+      <origin xyz="0 0 0" rpy="0 1.5708 0"/>
+      <geometry>
+        <cylinder radius="0.3425" length="0.22"/>
       </geometry>
     </collision>

Commit message: Remove tags unnecessary for libgazebo_ros_ackermann_drive.so

File: description/urdf/autocar_core.xacro (robot description, xacro)
@@ -186,5 +186,4 @@
     </inertial>
   </link>
-  <link name="steering_wheel" />  <!-- FIXME: missing inertia, error in rviz2 -->
   <joint name="br_axle" type="continuous">
     <origin rpy="0 0 0" xyz="0.8750 -1.013637 -0.144363" />
@@ -227,11 +226,4 @@
     <limit effort="1000.0" lower="-0.95" upper="0.95" velocity="100" />
   </joint>
-  <joint name="steering_joint" type="revolute">
-    <origin rpy="-0.002 0 0" xyz="0 0 0" />
-    <parent link="chassis_link" />
-    <child link="steering_wheel" />
-    <axis xyz="-0.964118 0.000768 0.265556" />
-    <limit effort="1000.0" lower="-100" upper="100" velocity="100" />
-  </joint>
   <gazebo reference="chassis_link">
     <material>Gazebo/White</material>
@@ -268,6 +260,6 @@
   <gazebo reference="fl_1">
     <material>Gazebo/DarkGrey</material>
-    <mu1>1.1</mu1>
-    <mu2>1.1</mu2>
+    <mu1>1.7</mu1>
+    <mu2>1.7</mu2>
     <selfCollide>true</selfCollide>
   </gazebo>

File: description/urdf/autocar_gazebo_control.xacro (robot description, xacro)
@@ -3,9 +3,10 @@
   <gazebo>
     <plugin name="ackermann_drive" filename="libgazebo_ros_ackermann_drive.so">
-      <ros>
+      <!-- <ros>
+        <namespace>autocar</namespace>
         <remapping>cmd_vel:=cmd_vel</remapping>
         <remapping>odom:=odom</remapping>
         <remapping>distance:=distance</remapping>
-      </ros>
+      </ros> -->
       <update_rate>100.0</update_rate>
       <!-- wheels -->
@@ -16,10 +17,10 @@
       <left_steering_joint>l_steer</left_steering_joint>
       <right_steering_joint>r_steer</right_steering_joint>
-      <steering_wheel_joint>steering_joint</steering_wheel_joint>
+      <!-- <steering_wheel_joint>steering_joint</steering_wheel_joint> -->
       <!-- Max absolute steer angle for tyre in radians-->
       <!-- Any cmd_vel angular z greater than this would be capped -->
       <max_steer>0.85</max_steer>
       <!-- Max absolute steering angle of steering wheel -->
-      <max_steering_angle>7.85</max_steering_angle>
+      <!-- <max_steering_angle>7.85</max_steering_angle> -->
       <!-- Max absolute linear speed in m/s -->
       <max_speed>20</max_speed>

Commit message: Revise urdf to comply with coordinate orientation convention

File: description/urdf/autocar_core.xacro (robot description, xacro)
@@ -17,5 +17,5 @@
   <joint name="hokuyo_joint" type="fixed">
     <axis xyz="0 1 0" />
-    <origin xyz="0 2.34 0.24" rpy="0 0 1.5708" />
+    <origin xyz="2.34 0 0.24" rpy="0 0 0" />
     <parent link="chassis_link" />
     <child link="hokuyo_link" />
@@ -23,5 +23,5 @@
   <link name="hokuyo_link">
     <collision>
-      <origin xyz="0 0 0" rpy="0 0 1.0" />
+      <origin xyz="0 0 0" rpy="0 0 0" />
       <geometry>
         <box size="0.05 0.05 0.05" />
@@ -42,10 +42,10 @@
   <link name="chassis_link">
     <inertial>
-      <origin rpy="0 0 0" xyz="1.04282e-06 0.07307 0.1816" />
+      <origin rpy="0 0 0" xyz="0.07307 1.04282e-06 0.1816" />
       <mass value="1580" />
-      <inertia ixx="1997.8579" ixy="-3e-05" ixz="-1e-06" iyy="442.7692" iyz="62.5206" izz="2238.0524" />
-    </inertial>
-    <visual>
-      <origin rpy="0 0 0" xyz="0 0 0" />
+      <inertia ixx="442.7692" ixy="3e-05" ixz="62.5206" iyy="1997.8579" iyz="1e-06" izz="2238.0524" />
+    </inertial>
+    <visual>
+      <origin rpy="0 0 -1.5708" xyz="0 0 0" />
       <geometry>
         <mesh filename="file://$(find description)/meshes/chassis_link.stl" scale="0.001 0.001 0.001" />
@@ -54,5 +54,5 @@
     </visual>
     <collision>
-      <origin rpy="0 0 0" xyz="0 0 0" />
+      <origin rpy="0 0 -1.5708" xyz="0 0 0" />
       <geometry>
         <mesh filename="file://$(find description)/meshes/chassis_link.stl" scale="0.001 0.001 0.001" />
@@ -61,5 +61,5 @@
   </link>
   <joint name="spoiler_joint" type="fixed">
-    <origin xyz="0 0.05 -0.05" rpy="1.5708 0 3.14159" />
+    <origin xyz="0.05 0 -0.05" rpy="0 0 0" />
     <parent link="chassis_link" />
     <child link="spoiler_link" />
@@ -67,5 +67,5 @@
   <link name="spoiler_link">
     <visual>
-      <origin rpy="0 0 0" xyz="0 0 0" />
+      <origin rpy="1.5708 0 1.5708" xyz="0 0 0" />
       <geometry>
         <mesh filename="file://$(find description)/meshes/spoiler.stl" scale="0.001 0.001 0.001" />
@@ -74,5 +74,5 @@
     </visual>
     <collision>
-      <origin rpy="0 0 0" xyz="0 0 0" />
+      <origin rpy="1.5708 0 1.5708" xyz="0 0 0" />
       <geometry>
         <mesh filename="file://$(find description)/meshes/spoiler.stl" scale="0.001 0.001 0.001" />
@@ -83,10 +83,10 @@
   <link name="br_1">
     <inertial>
-      <origin rpy="0 0 0" xyz="-0.0377 1.5929e-07 -1.5929e-07" />
-      <mass value="24.5" />
-      <inertia ixx="1.845139" ixy="-0.0" ixz="-0.0" iyy="1.049606" iyz="0.0" izz="1.049606" />
-    </inertial>
-    <visual>
-      <origin rpy="0 0 0" xyz="-0.8750 1.0136 0.1444" />
+      <origin rpy="0 0 -1.5708" xyz="1.5929e-07 0.0377 -1.5929e-07" />
+      <mass value="24.5" />
+      <inertia ixx="1.049606" ixy="0.0" ixz="0.0" iyy="1.845139" iyz="0.0" izz="1.049606" />
+    </inertial>
+    <visual>
+      <origin rpy="0 0 -1.5708" xyz="1.0136 0.8750 0.1444" />
       <geometry>
         <mesh filename="file://$(find description)/meshes/br_1.stl" scale="0.001 0.001 0.001" />
@@ -101,5 +101,5 @@
       </geometry>
       -->
-      <origin xyz="0 0 0" rpy="0 1.5708 0"/>
+      <origin xyz="0 0 0" rpy="1.5708 0 0"/>
       <geometry>
         <cylinder radius="0.3425" length="0.22"/>
@@ -109,10 +109,10 @@
   <link name="bl_1">
     <inertial>
-      <origin rpy="0 0 0" xyz="-0.0377 1.5929e-07 -1.5929e-07" />
-      <mass value="24.5" />
-      <inertia ixx="1.845139" ixy="-0.0" ixz="-0.0" iyy="1.049606" iyz="0.0" izz="1.049606" />
-    </inertial>
-    <visual>
-      <origin rpy="0 0 0" xyz="0.8750 1.0136 0.1444" />
+      <origin rpy="0 0 -1.5708" xyz="1.5929e-07 -0.0377 -1.5929e-07" />
+      <mass value="24.5" />
+      <inertia ixx="1.049606" ixy="0.0" ixz="0.0" iyy="1.845139" iyz="0.0" izz="1.049606" />
+    </inertial>
+    <visual>
+      <origin rpy="0 0 -1.5708" xyz="1.0136 -0.8750 0.1444" />
       <geometry>
         <mesh filename="file://$(find description)/meshes/bl_1.stl" scale="0.001 0.001 0.001" />
@@ -127,5 +127,5 @@
       </geometry>
       -->
-      <origin xyz="0 0 0" rpy="0 1.5708 0"/>
+      <origin xyz="0 0 0" rpy="1.5708 0 0"/>
       <geometry>
         <cylinder radius="0.3425" length="0.22"/>
@@ -135,10 +135,10 @@
   <link name="fr_1">
     <inertial>
-      <origin rpy="0 0 0" xyz="-0.0377 1.5929e-07 -1.5929e-07" />
-      <mass value="24.5" />
-      <inertia ixx="1.845139" ixy="-0.0" ixz="-0.0" iyy="1.049606" iyz="0.0" izz="1.049606" />
-    </inertial>
-    <visual>
-      <origin rpy="0 0 0" xyz="-0.8750 -1.5174 0.1444" />
+      <origin rpy="0 0 -1.5708" xyz="1.5929e-07 0.0377 -1.5929e-07" />
+      <mass value="24.5" />
+      <inertia ixx="1.049606" ixy="-0.0" ixz="0.0" iyy="1.845139" iyz="0.0" izz="1.049606" />
+    </inertial>
+    <visual>
+      <origin rpy="0 0 -1.5708" xyz="-1.5174 0.8750 0.1444" />
       <geometry>
         <mesh filename="file://$(find description)/meshes/fr_1.stl" scale="0.001 0.001 0.001" />
@@ -147,5 +147,5 @@
     </visual>
     <collision>
-      <origin rpy="0 0 0" xyz="-0.8750 -1.5174 0.1444" />
+      <origin rpy="0 0 -1.5708" xyz="-1.5174 0.8750 0.1444" />
       <geometry>
         <mesh filename="file://$(find description)/meshes/fr_1.stl" scale="0.001 0.001 0.001" />
@@ -155,10 +155,10 @@
   <link name="fl_1">
     <inertial>
-      <origin rpy="0 0 0" xyz="-0.0377 1.5929e-07 -1.5929e-07" />
-      <mass value="24.5" />
-      <inertia ixx="1.845139" ixy="-0.0" ixz="-0.0" iyy="1.049606" iyz="0.0" izz="1.049606" />
-    </inertial>
-    <visual>
-      <origin rpy="0 0 0" xyz="0.8750 -1.5174 0.1444" />
+      <origin rpy="0 0 -1.5708" xyz="1.5929e-07 -0.0377 -1.5929e-07" />
+      <mass value="24.5" />
+      <inertia ixx="1.049606" ixy="0.0" ixz="0.0" iyy="1.845139" iyz="0.0" izz="1.049606" />
+    </inertial>
+    <visual>
+      <origin rpy="0 0 -1.5708" xyz="-1.5174 -0.8750 0.1444" />
       <geometry>
         <mesh filename="file://$(find description)/meshes/fl_1.stl" scale="0.001 0.001 0.001" />
@@ -167,5 +167,5 @@
     </visual>
     <collision>
-      <origin rpy="0 0 0" xyz="0.8750 -1.5174 0.1444" />
+      <origin rpy="0 0 -1.5708" xyz="-1.5174 -0.8750 0.1444" />
       <geometry>
         <mesh filename="file://$(find description)/meshes/fl_1.stl" scale="0.001 0.001 0.001" />
@@ -175,5 +175,5 @@
   <link name="r_steer_1">
     <inertial>
-      <origin rpy="0 0 0" xyz="0.003381 1.5929e-07 0.02162" />
+      <origin rpy="0 0 0" xyz="1.5929e-07 -0.003381 0.02162" />
       <mass value="1" />
       <inertia ixx="1.0" ixy="0.0" ixz="0.0" iyy="1.0" iyz="0.0" izz="1.0" />
@@ -182,5 +182,5 @@
   <link name="l_steer_1">
     <inertial>
-      <origin rpy="0 0 0" xyz="0.003381 1.5929e-07 0.02162" />
+      <origin rpy="0 0 0" xyz="1.5929e-07 0.003381 0.02162" />
       <mass value="1" />
       <inertia ixx="1.0" ixy="0.0" ixz="0.0" iyy="1.0" iyz="0.0" izz="1.0" />
@@ -188,29 +188,29 @@
   </link>
   <joint name="br_axle" type="continuous">
-    <origin rpy="0 0 0" xyz="0.8750 -1.013637 -0.144363" />
+    <origin rpy="0 0 0" xyz="-1.013637 -0.8750 -0.144363" />
     <parent link="chassis_link" />
     <child link="br_1" />
-    <axis xyz="-1.0 0.0 0.0" />
+    <axis xyz="0.0 1.0 0.0" />
   </joint>
   <joint name="bl_axle" type="continuous">
-    <origin rpy="0 0 0" xyz="-0.8750 -1.013637 -0.144363" />
+    <origin rpy="0 0 0" xyz="-1.013637 0.8750 -0.144363" />
     <parent link="chassis_link" />
     <child link="bl_1" />
-    <axis xyz="-1.0 0.0 0.0" />
+    <axis xyz="0.0 1.0 0.0" />
   </joint>
   <joint name="fr_axle" type="continuous">
-    <origin rpy="0 0 0" xyz="0.05 0.0 0.0" />
+    <origin rpy="0 0 0" xyz="0.0 -0.05 0.0" />
     <parent link="r_steer_1" />
     <child link="fr_1" />
-    <axis xyz="-1.0 0.0 0.0" />
+    <axis xyz="0.0 1.0 0.0" />
   </joint>
   <joint name="fl_axle" type="continuous">
-    <origin rpy="0 0 0" xyz="-0.05 0.0 0.0" />
+    <origin rpy="0 0 0" xyz="0.0 0.05 0.0" />
     <parent link="l_steer_1" />
     <child link="fl_1" />
-    <axis xyz="-1.0 0.0 0.0" />
+    <axis xyz="0.0 1.0 0.0" />
   </joint>
   <joint name="r_steer" type="revolute">
-    <origin rpy="0 0 0" xyz="0.8250 1.517363 -0.144363" />
+    <origin rpy="0 0 0" xyz="1.517363 -0.8250 -0.144363" />
     <parent link="chassis_link" />
     <child link="r_steer_1" />
@@ -220,5 +220,5 @@
   </joint>
   <joint name="l_steer" type="revolute">
-    <origin rpy="0 0 0" xyz="-0.8250 1.517363 -0.144363" />
+    <origin rpy="0 0 0" xyz="1.517363 0.8250 -0.144363" />
     <parent link="chassis_link" />
     <child link="l_steer_1" />

Commit message: Make wheel as sphere

File: description/urdf/autocar_core.xacro (robot description, xacro)
@@ -103,5 +103,5 @@
       <origin xyz="0 0 0" rpy="1.5708 0 0"/>
       <geometry>
-        <cylinder radius="0.3425" length="0.22"/>
+        <sphere radius="0.3425"/>
       </geometry>
     </collision>
@@ -129,5 +129,5 @@
       <origin xyz="0 0 0" rpy="1.5708 0 0"/>
       <geometry>
-        <cylinder radius="0.3425" length="0.22"/>
+        <sphere radius="0.3425"/>
       </geometry>
     </collision>
@@ -147,7 +147,7 @@
     </visual>
     <collision>
-      <origin rpy="0 0 -1.5708" xyz="-1.5174 0.8750 0.1444" />
-      <geometry>
-        <mesh filename="file://$(find description)/meshes/fr_1.stl" scale="0.001 0.001 0.001" />
+      <origin xyz="0 0 0" rpy="1.5708 0 0"/>
+      <geometry>
+        <sphere radius="0.3425"/>
       </geometry>
     </collision>
@@ -167,7 +167,7 @@
     </visual>
     <collision>
-      <origin rpy="0 0 -1.5708" xyz="-1.5174 -0.8750 0.1444" />
-      <geometry>
-        <mesh filename="file://$(find description)/meshes/fl_1.stl" scale="0.001 0.001 0.001" />
+      <origin xyz="0 0 0" rpy="1.5708 0 0"/>
+      <geometry>
+        <sphere radius="0.3425"/>
       </geometry>
     </collision>

Commit message: Increase steering damping

File: description/urdf/autocar_core.xacro (robot description, xacro)
@@ -80,5 +80,5 @@
     </collision>
   </link>
-  <!-- ALC231031 - TODO - Revise friction, dynamics, dampling, slides, shere wheel, etc. -->
+  <!-- ALC231031 - TODO - Revise friction, dynamics, slides, etc. -->
   <link name="br_1">
     <inertial>
@@ -216,5 +216,5 @@
     <child link="r_steer_1" />
     <axis xyz="0.0 0.0 1.0" />
-    <dynamics damping="0.01" friction="0.01" />
+    <dynamics damping="50.0" friction="0.01" />
     <limit effort="1000.0" lower="-0.95" upper="0.95" velocity="100" />
   </joint>
@@ -224,5 +224,5 @@
     <child link="l_steer_1" />
     <axis xyz="0.0 0.0 1.0" />
-    <dynamics damping="0.01" friction="0.01" />
+    <dynamics damping="50.0" friction="0.01" />
     <limit effort="1000.0" lower="-0.95" upper="0.95" velocity="100" />
   </joint>

Commit message: Revise inertia to reduce slipping effect of the front wheels

File: description/urdf/autocar_core.xacro (robot description, xacro)
@@ -85,5 +85,5 @@
       <origin rpy="0 0 -1.5708" xyz="1.5929e-07 0.0377 -1.5929e-07" />
       <mass value="24.5" />
-      <inertia ixx="1.049606" ixy="0.0" ixz="0.0" iyy="1.845139" iyz="0.0" izz="1.049606" />
+      <inertia ixx="1.845139" ixy="0.0" ixz="0.0" iyy="1.049606" iyz="0.0" izz="1.049606" />
     </inertial>
     <visual>
@@ -111,5 +111,5 @@
       <origin rpy="0 0 -1.5708" xyz="1.5929e-07 -0.0377 -1.5929e-07" />
       <mass value="24.5" />
-      <inertia ixx="1.049606" ixy="0.0" ixz="0.0" iyy="1.845139" iyz="0.0" izz="1.049606" />
+      <inertia ixx="1.845139" ixy="0.0" ixz="0.0" iyy="1.049606" iyz="0.0" izz="1.049606" />
     </inertial>
     <visual>
@@ -137,5 +137,5 @@
       <origin rpy="0 0 -1.5708" xyz="1.5929e-07 0.0377 -1.5929e-07" />
       <mass value="24.5" />
-      <inertia ixx="1.049606" ixy="-0.0" ixz="0.0" iyy="1.845139" iyz="0.0" izz="1.049606" />
+      <inertia ixx="0.01845139" ixy="0.0" ixz="0.0" iyy="0.01049606" iyz="0.0" izz="0.01049606" />
     </inertial>
     <visual>
@@ -157,5 +157,5 @@
       <origin rpy="0 0 -1.5708" xyz="1.5929e-07 -0.0377 -1.5929e-07" />
       <mass value="24.5" />
-      <inertia ixx="1.049606" ixy="0.0" ixz="0.0" iyy="1.845139" iyz="0.0" izz="1.049606" />
+      <inertia ixx="0.01845139" ixy="0.0" ixz="0.0" iyy="0.01049606" iyz="0.0" izz="0.01049606" />
     </inertial>
     <visual>
@@ -177,5 +177,5 @@
       <origin rpy="0 0 0" xyz="1.5929e-07 -0.003381 0.02162" />
       <mass value="1" />
-      <inertia ixx="1.0" ixy="0.0" ixz="0.0" iyy="1.0" iyz="0.0" izz="1.0" />
+      <inertia ixx="0.14583300" ixy="0.0" ixz="0.0" iyy="0.14583300" iyz="0.0" izz="0.12500000" />
     </inertial>
   </link>
@@ -184,5 +184,5 @@
       <origin rpy="0 0 0" xyz="1.5929e-07 0.003381 0.02162" />
       <mass value="1" />
-      <inertia ixx="1.0" ixy="0.0" ixz="0.0" iyy="1.0" iyz="0.0" izz="1.0" />
+      <inertia ixx="0.14583300" ixy="0.0" ixz="0.0" iyy="0.14583300" iyz="0.0" izz="0.12500000" />
     </inertial>
   </link>
