Commit message: Fix "unable to spawn meshes into gazebo", by not using package://package_name in <mesh filename=.../>, and use file://$(find package_name) instead

File: description/urdf/autocar.urdf.xacro (robot description, xacro)
@@ -31,5 +31,5 @@
       <origin xyz="0 0 0" rpy="0 0 0" />
       <geometry>
-        <mesh filename="package://description/meshes/hokuyo.dae" />
+        <mesh filename="file://$(find description)/meshes/hokuyo.dae" />
       </geometry>
     </visual>
@@ -49,5 +49,5 @@
       <origin rpy="0 0 0" xyz="0 0 0" />
       <geometry>
-        <mesh filename="package://description/meshes/chassis_link.stl" scale="0.001 0.001 0.001" />
+        <mesh filename="file://$(find description)/meshes/chassis_link.stl" scale="0.001 0.001 0.001" />
       </geometry>
       <material name="silver" />
@@ -56,5 +56,5 @@
       <origin rpy="0 0 0" xyz="0 0 0" />
       <geometry>
-        <mesh filename="package://description/meshes/chassis_link.stl" scale="0.001 0.001 0.001" />
+        <mesh filename="file://$(find description)/meshes/chassis_link.stl" scale="0.001 0.001 0.001" />
       </geometry>
     </collision>
@@ -69,5 +69,5 @@
       <origin rpy="0 0 0" xyz="0 0 0" />
       <geometry>
-        <mesh filename="package://description/meshes/spoiler.stl" scale="0.001 0.001 0.001" />
+        <mesh filename="file://$(find description)/meshes/spoiler.stl" scale="0.001 0.001 0.001" />
       </geometry>
       <material name="silver" />
@@ -76,5 +76,5 @@
       <origin rpy="0 0 0" xyz="0 0 0" />
       <geometry>
-        <mesh filename="package://description/meshes/spoiler.stl" scale="0.001 0.001 0.001" />
+        <mesh filename="file://$(find description)/meshes/spoiler.stl" scale="0.001 0.001 0.001" />
       </geometry>
     </collision>
@@ -89,5 +89,5 @@
       <origin rpy="0 0 0" xyz="-0.8750 1.0136 0.1444" />
       <geometry>
-        <mesh filename="package://description/meshes/br_1.stl" scale="0.001 0.001 0.001" />
+        <mesh filename="file://$(find description)/meshes/br_1.stl" scale="0.001 0.001 0.001" />
       </geometry>
       <material name="darkgrey" />
@@ -96,5 +96,5 @@
       <origin rpy="0 0 0" xyz="-0.8750 1.0136 0.1444" />
       <geometry>
-        <mesh filename="package://description/meshes/br_1.stl" scale="0.001 0.001 0.001" />
+        <mesh filename="file://$(find description)/meshes/br_1.stl" scale="0.001 0.001 0.001" />
       </geometry>
     </collision>
@@ -109,5 +109,5 @@
       <origin rpy="0 0 0" xyz="0.8750 1.0136 0.1444" />
       <geometry>
-        <mesh filename="package://description/meshes/bl_1.stl" scale="0.001 0.001 0.001" />
+        <mesh filename="file://$(find description)/meshes/bl_1.stl" scale="0.001 0.001 0.001" />
       </geometry>
       <material name="darkgrey" />
@@ -116,5 +116,5 @@
       <origin rpy="0 0 0" xyz="0.8750 1.0136 0.1444" />
       <geometry>
-        <mesh filename="package://description/meshes/bl_1.stl" scale="0.001 0.001 0.001" />
+        <mesh filename="file://$(find description)/meshes/bl_1.stl" scale="0.001 0.001 0.001" />
       </geometry>
     </collision>
@@ -129,5 +129,5 @@
       <origin rpy="0 0 0" xyz="-0.8750 -1.5174 0.1444" />
       <geometry>
-        <mesh filename="package://description/meshes/fr_1.stl" scale="0.001 0.001 0.001" />
+        <mesh filename="file://$(find description)/meshes/fr_1.stl" scale="0.001 0.001 0.001" />
       </geometry>
       <material name="darkgrey" />
@@ -136,5 +136,5 @@
       <origin rpy="0 0 0" xyz="-0.8750 -1.5174 0.1444" />
       <geometry>
-        <mesh filename="package://description/meshes/fr_1.stl" scale="0.001 0.001 0.001" />
+        <mesh filename="file://$(find description)/meshes/fr_1.stl" scale="0.001 0.001 0.001" />
       </geometry>
     </collision>
@@ -149,5 +149,5 @@
       <origin rpy="0 0 0" xyz="0.8750 -1.5174 0.1444" />
       <geometry>
-        <mesh filename="package://description/meshes/fl_1.stl" scale="0.001 0.001 0.001" />
+        <mesh filename="file://$(find description)/meshes/fl_1.stl" scale="0.001 0.001 0.001" />
       </geometry>
       <material name="darkgrey" />
@@ -156,5 +156,5 @@
       <origin rpy="0 0 0" xyz="0.8750 -1.5174 0.1444" />
       <geometry>
-        <mesh filename="package://description/meshes/fl_1.stl" scale="0.001 0.001 0.001" />
+        <mesh filename="file://$(find description)/meshes/fl_1.stl" scale="0.001 0.001 0.001" />
       </geometry>
     </collision>

Commit message: FIXME: gazebo_ros_ackermann_drive can publish joint_state but no response to cmd_vel control fron teleop_twist_keyboard by `ros2 run teleop_twist_keyboard teleop_twist_keyboard`

File: description/urdf/autocar.urdf.xacro (robot description, xacro)
@@ -1,266 +1,5 @@
 <?xml version="1.0"?>
 <robot name="autocar" xmlns:xacro="http://www.ros.org/wiki/xacro">
-  <!-- RVIZ MATERIAL COLOUR -->
-  <material name="silver">
-    <color rgba="0.1 0.1 0.1 0.5" />
-  </material>
-  <material name="darkgrey">
-    <color rgba="0 0 0 0.7" />
-  </material>
-  <!-- ROBOT DEFINITION -->
-  <link name="base_link" />
-  <joint name="chassis_link_joint" type="fixed">
-    <origin xyz="0 0 0.4936" rpy="0 0 0" />
-    <parent link="base_link" />
-    <child link="chassis_link" />
-  </joint>
-  <joint name="hokuyo_joint" type="fixed">
-    <axis xyz="0 1 0" />
-    <origin xyz="0 2.34 0.24" rpy="0 0 1.5708" />
-    <parent link="chassis_link" />
-    <child link="hokuyo_link" />
-  </joint>
-  <link name="hokuyo_link">
-    <collision>
-      <origin xyz="0 0 0" rpy="0 0 1.0" />
-      <geometry>
-        <box size="0.05 0.05 0.05" />
-      </geometry>
-    </collision>
-    <visual>
-      <origin xyz="0 0 0" rpy="0 0 0" />
-      <geometry>
-        <mesh filename="file://$(find description)/meshes/hokuyo.dae" />
-      </geometry>
-    </visual>
-    <inertial>
-      <mass value="1e-5" />
-      <origin xyz="0 0 0" rpy="0 0 0" />
-      <inertia ixx="1e-6" ixy="0" ixz="0" iyy="1e-6" iyz="0" izz="1e-6" />
-    </inertial>
-  </link>
-  <link name="chassis_link">
-    <inertial>
-      <origin rpy="0 0 0" xyz="1.04282e-06 0.07307 0.1816" />
-      <mass value="1580" />
-      <inertia ixx="1997.8579" ixy="-3e-05" ixz="-1e-06" iyy="442.7692" iyz="62.5206" izz="2238.0524" />
-    </inertial>
-    <visual>
-      <origin rpy="0 0 0" xyz="0 0 0" />
-      <geometry>
-        <mesh filename="file://$(find description)/meshes/chassis_link.stl" scale="0.001 0.001 0.001" />
-      </geometry>
-      <material name="silver" />
-    </visual>
-    <collision>
-      <origin rpy="0 0 0" xyz="0 0 0" />
-      <geometry>
-        <mesh filename="file://$(find description)/meshes/chassis_link.stl" scale="0.001 0.001 0.001" />
-      </geometry>
-    </collision>
-  </link>
-  <joint name="spoiler_joint" type="fixed">
-    <origin xyz="0 0.05 -0.05" rpy="1.5708 0 3.14159" />
-    <parent link="chassis_link" />
-    <child link="spoiler_link" />
-  </joint>
-  <link name="spoiler_link">
-    <visual>
-      <origin rpy="0 0 0" xyz="0 0 0" />
-      <geometry>
-        <mesh filename="file://$(find description)/meshes/spoiler.stl" scale="0.001 0.001 0.001" />
-      </geometry>
-      <material name="silver" />
-    </visual>
-    <collision>
-      <origin rpy="0 0 0" xyz="0 0 0" />
-      <geometry>
-        <mesh filename="file://$(find description)/meshes/spoiler.stl" scale="0.001 0.001 0.001" />
-      </geometry>
-    </collision>
-  </link>
-  <link name="br_1">
-    <inertial>
-      <origin rpy="0 0 0" xyz="-0.0377 1.5929e-07 -1.5929e-07" />
-      <mass value="24.5" />
-      <inertia ixx="1.845139" ixy="-0.0" ixz="-0.0" iyy="1.049606" iyz="0.0" izz="1.049606" />
-    </inertial>
-    <visual>
-      <origin rpy="0 0 0" xyz="-0.8750 1.0136 0.1444" />
-      <geometry>
-        <mesh filename="file://$(find description)/meshes/br_1.stl" scale="0.001 0.001 0.001" />
-      </geometry>
-      <material name="darkgrey" />
-    </visual>
-    <collision>
-      <origin rpy="0 0 0" xyz="-0.8750 1.0136 0.1444" />
-      <geometry>
-        <mesh filename="file://$(find description)/meshes/br_1.stl" scale="0.001 0.001 0.001" />
-      </geometry>
-    </collision>
-  </link>
-  <link name="bl_1">
-    <inertial>
-      <origin rpy="0 0 0" xyz="-0.0377 1.5929e-07 -1.5929e-07" />
-      <mass value="24.5" />
-      <inertia ixx="1.845139" ixy="-0.0" ixz="-0.0" iyy="1.049606" iyz="0.0" izz="1.049606" />
-    </inertial>
-    <visual>
-      <origin rpy="0 0 0" xyz="0.8750 1.0136 0.1444" />
-      <geometry>
-        <mesh filename="file://$(find description)/meshes/bl_1.stl" scale="0.001 0.001 0.001" />
-      </geometry>
-      <material name="darkgrey" />
-    </visual>
-    <collision>
-      <origin rpy="0 0 0" xyz="0.8750 1.0136 0.1444" />
-      <geometry>
-        <mesh filename="file://$(find description)/meshes/bl_1.stl" scale="0.001 0.001 0.001" />
-      </geometry>
-    </collision>
-  </link>
-  <link name="fr_1">
-    <inertial>
-      <origin rpy="0 0 0" xyz="-0.0377 1.5929e-07 -1.5929e-07" />
-      <mass value="24.5" />
-      <inertia ixx="1.845139" ixy="-0.0" ixz="-0.0" iyy="1.049606" iyz="0.0" izz="1.049606" />
-    </inertial>
-    <visual>
-      <origin rpy="0 0 0" xyz="-0.8750 -1.5174 0.1444" />
-      <geometry>
-        <mesh filename="file://$(find description)/meshes/fr_1.stl" scale="0.001 0.001 0.001" />
-      </geometry>
-      <material name="darkgrey" />
-    </visual>
-    <collision>
-      <origin rpy="0 0 0" xyz="-0.8750 -1.5174 0.1444" />
-      <geometry>
-        <mesh filename="file://$(find description)/meshes/fr_1.stl" scale="0.001 0.001 0.001" />
-      </geometry>
-    </collision>
-  </link>
-  <link name="fl_1">
-    <inertial>
-      <origin rpy="0 0 0" xyz="-0.0377 1.5929e-07 -1.5929e-07" />
-      <mass value="24.5" />
-      <inertia ixx="1.845139" ixy="-0.0" ixz="-0.0" iyy="1.049606" iyz="0.0" izz="1.049606" />
-    </inertial>
-    <visual>
-      <origin rpy="0 0 0" xyz="0.8750 -1.5174 0.1444" />
-      <geometry>
-        <mesh filename="file://$(find description)/meshes/fl_1.stl" scale="0.001 0.001 0.001" />
-      </geometry>
-      <material name="darkgrey" />
-    </visual>
-    <collision>
-      <origin rpy="0 0 0" xyz="0.8750 -1.5174 0.1444" />
-      <geometry>
-        <mesh filename="file://$(find description)/meshes/fl_1.stl" scale="0.001 0.001 0.001" />
-      </geometry>
-    </collision>
-  </link>
-  <link name="r_steer_1">
-    <inertial>
-      <origin rpy="0 0 0" xyz="0.003381 1.5929e-07 0.02162" />
-      <mass value="1" />
-      <inertia ixx="1.0" ixy="0.0" ixz="0.0" iyy="1.0" iyz="0.0" izz="1.0" />
-    </inertial>
-  </link>
-  <link name="l_steer_1">
-    <inertial>
-      <origin rpy="0 0 0" xyz="0.003381 1.5929e-07 0.02162" />
-      <mass value="1" />
-      <inertia ixx="1.0" ixy="0.0" ixz="0.0" iyy="1.0" iyz="0.0" izz="1.0" />
-    </inertial>
-  </link>
-  <joint name="br_axle" type="continuous">
-    <origin rpy="0 0 0" xyz="0.8750 -1.013637 -0.144363" />
-    <parent link="chassis_link" />
-    <child link="br_1" />
-    <axis xyz="-1.0 0.0 0.0" />
-  </joint>
-  <joint name="bl_axle" type="continuous">
-    <origin rpy="0 0 0" xyz="-0.8750 -1.013637 -0.144363" />
-    <parent link="chassis_link" />
-    <child link="bl_1" />
-    <axis xyz="-1.0 0.0 0.0" />
-  </joint>
-  <joint name="fr_axle" type="continuous">
-    <origin rpy="0 0 0" xyz="0.05 0.0 0.0" />
-    <parent link="r_steer_1" />
-    <child link="fr_1" />
-    <axis xyz="-1.0 0.0 0.0" />
-  </joint>
-  <joint name="fl_axle" type="continuous">
-    <origin rpy="0 0 0" xyz="-0.05 0.0 0.0" />
-    <parent link="l_steer_1" />
-    <child link="fl_1" />
-    <axis xyz="-1.0 0.0 0.0" />
-  </joint>
-  <joint name="r_steer" type="revolute">
-    <origin rpy="0 0 0" xyz="0.8250 1.517363 -0.144363" />
-    <parent link="chassis_link" />
-    <child link="r_steer_1" />
-    <axis xyz="0.0 0.0 1.0" />
-    <dynamics damping="0.01" friction="0.01" />
-    <limit effort="1000.0" lower="-0.95" upper="0.95" velocity="100" />
-  </joint>
-  <joint name="l_steer" type="revolute">
-    <origin rpy="0 0 0" xyz="-0.8250 1.517363 -0.144363" />
-    <parent link="chassis_link" />
-    <child link="l_steer_1" />
-    <axis xyz="0.0 0.0 1.0" />
-    <dynamics damping="0.01" friction="0.01" />
-    <limit effort="1000.0" lower="-0.95" upper="0.95" velocity="100" />
-  </joint>
-  <gazebo reference="chassis_link">
-    <material>Gazebo/White</material>
-    <mu1>0.2</mu1>
-    <mu2>0.2</mu2>
-    <selfCollide>true</selfCollide>
-    <gravity>true</gravity>
-  </gazebo>
-  <gazebo reference="spoiler_link">
-    <material>Gazebo/DarkGrey</material>
-    <mu1>0.2</mu1>
-    <mu2>0.2</mu2>
-    <selfCollide>true</selfCollide>
-    <gravity>true</gravity>
-  </gazebo>
-  <gazebo reference="br_1">
-    <material>Gazebo/DarkGrey</material>
-    <mu1>1.7</mu1>
-    <mu2>1.7</mu2>
-    <selfCollide>true</selfCollide>
-  </gazebo>
-  <gazebo reference="bl_1">
-    <material>Gazebo/DarkGrey</material>
-    <mu1>1.7</mu1>
-    <mu2>1.7</mu2>
-    <selfCollide>true</selfCollide>
-  </gazebo>
-  <gazebo reference="fr_1">
-    <material>Gazebo/DarkGrey</material>
-    <mu1>1.7</mu1>
-    <mu2>1.7</mu2>
-    <selfCollide>true</selfCollide>
-  </gazebo>
-  <gazebo reference="fl_1">
-    <material>Gazebo/DarkGrey</material>
-    <mu1>1.1</mu1>
-    <mu2>1.1</mu2>
-    <selfCollide>true</selfCollide>
-  </gazebo>
-  <gazebo reference="r_steer_1">
-    <material>Gazebo/DarkGrey</material>
-    <mu1>0.2</mu1>
-    <mu2>0.2</mu2>
-    <selfCollide>true</selfCollide>
-  </gazebo>
-  <gazebo reference="l_steer_1">
-    <material>Gazebo/DarkGrey</material>
-    <mu1>0.2</mu1>
-    <mu2>0.2</mu2>
-    <selfCollide>true</selfCollide>
-  </gazebo>
+  <xacro:include filename="autocar_core.xacro" />
+  <xacro:include filename="autocar_gazebo_control.xacro" />
 </robot>

Commit message: Add rear-wheel steer

File: description/urdf/autocar.urdf.xacro (robot description, xacro)
@@ -1,4 +1,5 @@
 <?xml version="1.0"?>
 <robot name="autocar" xmlns:xacro="http://www.ros.org/wiki/xacro">
+  <xacro:arg name="use_4ws" default="false"/>
   <xacro:arg name="use_ros2_control" default="false"/>
   <xacro:arg name="gazebo_control_config" default="autocar_ackermann_gazebo_control.xacro"/>

File: description/urdf/autocar_ackermann_gazebo_control.xacro (robot description, xacro)
@@ -15,6 +15,6 @@
       <rear_left_joint>bl_axle</rear_left_joint>
       <rear_right_joint>br_axle</rear_right_joint>
-      <left_steering_joint>l_steer</left_steering_joint>
-      <right_steering_joint>r_steer</right_steering_joint>
+      <left_steering_joint>fl_steer</left_steering_joint>
+      <right_steering_joint>fr_steer</right_steering_joint>
       <!-- <steering_wheel_joint>steering_joint</steering_wheel_joint> -->
       <!-- Max absolute steer angle for tyre in radians-->

File: description/urdf/autocar_core.xacro (robot description, xacro)
@@ -182,5 +182,5 @@
     </collision>
   </link>
-  <link name="r_steer_1">
+  <link name="fr_steer_1">
     <inertial>
       <origin rpy="0 0 0" xyz="0 0 0" />
@@ -189,5 +189,5 @@
     </inertial>
   </link>
-  <link name="l_steer_1">
+  <link name="fl_steer_1">
     <inertial>
       <origin rpy="0 0 0" xyz="0 0 0" />
@@ -196,13 +196,27 @@
     </inertial>
   </link>
+  <link name="br_steer_1">
+    <inertial>
+      <origin rpy="0 0 0" xyz="0 0 0" />
+      <mass value="1" />
+      <inertia ixx="0.004" ixy="0.0" ixz="0.0" iyy="0.004" iyz="0.0" izz="0.004"/>
+    </inertial>
+  </link>
+  <link name="bl_steer_1">
+    <inertial>
+      <origin rpy="0 0 0" xyz="0 0 0" />
+      <mass value="1" />
+      <inertia ixx="0.004" ixy="0.0" ixz="0.0" iyy="0.004" iyz="0.0" izz="0.004"/>
+    </inertial>
+  </link>
   <joint name="br_axle" type="continuous">
-    <origin rpy="0 0 0" xyz="-1.013637 -0.8750 -0.144363" />
-    <parent link="chassis_link" />
+    <origin rpy="0 0 0" xyz="0.0 0.0 0.0" />
+    <parent link="br_steer_1" />
     <child link="br_1" />
     <axis xyz="0.0 1.0 0.0" />
   </joint>
   <joint name="bl_axle" type="continuous">
-    <origin rpy="0 0 0" xyz="-1.013637 0.8750 -0.144363" />
-    <parent link="chassis_link" />
+    <origin rpy="0 0 0" xyz="0.0 0.0 0.0" />
+    <parent link="bl_steer_1" />
     <child link="bl_1" />
     <axis xyz="0.0 1.0 0.0" />
@@ -211,5 +225,5 @@
     <!-- NOTE - The key to avoid non-driven wheels split out is to make sure the steering joint is at the same location as the wheel rotation joint (or the center of mass of it). -->
     <origin rpy="0 0 0" xyz="0.0 0.0 0.0" />
-    <parent link="r_steer_1" />
+    <parent link="fr_steer_1" />
     <child link="fr_1" />
     <axis xyz="0.0 1.0 0.0" />
@@ -218,24 +232,60 @@
     <!-- NOTE - The key to avoid non-driven wheels split out is to make sure the steering joint is at the same location as the wheel rotation joint (or the center of mass of it). -->
     <origin rpy="0 0 0" xyz="0.0 0.0 0.0" />
-    <parent link="l_steer_1" />
+    <parent link="fl_steer_1" />
     <child link="fl_1" />
     <axis xyz="0.0 1.0 0.0" />
   </joint>
-  <joint name="r_steer" type="revolute">
+  <joint name="fr_steer" type="revolute">
     <origin rpy="0 0 0" xyz="1.517363 -0.8250 -0.144363" />
     <parent link="chassis_link" />
-    <child link="r_steer_1" />
+    <child link="fr_steer_1" />
     <axis xyz="0.0 0.0 1.0" />
     <dynamics damping="50.0" friction="0.01" />
     <limit effort="1000.0" lower="-0.95" upper="0.95" velocity="100" />
   </joint>
-  <joint name="l_steer" type="revolute">
+  <joint name="fl_steer" type="revolute">
     <origin rpy="0 0 0" xyz="1.517363 0.8250 -0.144363" />
     <parent link="chassis_link" />
-    <child link="l_steer_1" />
+    <child link="fl_steer_1" />
     <axis xyz="0.0 0.0 1.0" />
     <dynamics damping="50.0" friction="0.01" />
     <limit effort="1000.0" lower="-0.95" upper="0.95" velocity="100" />
   </joint>
+  <xacro:if value="$(arg use_4ws)">
+    <joint name="br_steer" type="revolute">
+      <origin rpy="0 0 0" xyz="-1.013637 -0.8750 -0.144363" />
+      <parent link="chassis_link" />
+      <child link="br_steer_1" />
+      <axis xyz="0.0 0.0 1.0" />
+      <dynamics damping="50.0" friction="0.01" />
+      <limit effort="1000.0" lower="-0.95" upper="0.95" velocity="100" />
+    </joint>
+    <joint name="bl_steer" type="revolute">
+      <origin rpy="0 0 0" xyz="-1.013637 0.8750 -0.144363" />
+      <parent link="chassis_link" />
+      <child link="bl_steer_1" />
+      <axis xyz="0.0 0.0 1.0" />
+      <dynamics damping="50.0" friction="0.01" />
+      <limit effort="1000.0" lower="-0.95" upper="0.95" velocity="100" />
+    </joint>
+  </xacro:if>
+  <xacro:unless value="$(arg use_4ws)">
+    <joint name="br_steer" type="fixed">
+      <origin rpy="0 0 0" xyz="-1.013637 -0.8750 -0.144363" />
+      <parent link="chassis_link" />
+      <child link="br_steer_1" />
+      <axis xyz="0.0 0.0 1.0" />
+      <dynamics damping="50.0" friction="0.01" />
+      <limit effort="1000.0" lower="-0.95" upper="0.95" velocity="100" />
+    </joint>
+    <joint name="bl_steer" type="fixed">
+      <origin rpy="0 0 0" xyz="-1.013637 0.8750 -0.144363" />
+      <parent link="chassis_link" />
+      <child link="bl_steer_1" />
+      <axis xyz="0.0 0.0 1.0" />
+      <dynamics damping="50.0" friction="0.01" />
+      <limit effort="1000.0" lower="-0.95" upper="0.95" velocity="100" />
+    </joint>
+  </xacro:unless>
   <gazebo reference="chassis_link">
     <material>Gazebo/White</material>
@@ -288,11 +338,23 @@
     <selfCollide>true</selfCollide>
   </gazebo>
-  <gazebo reference="r_steer_1">
-    <material>Gazebo/DarkGrey</material>
-    <mu1>0.2</mu1>
-    <mu2>0.2</mu2>
-    <selfCollide>true</selfCollide>
-  </gazebo>
-  <gazebo reference="l_steer_1">
+  <gazebo reference="fr_steer_1">
+    <material>Gazebo/DarkGrey</material>
+    <mu1>0.2</mu1>
+    <mu2>0.2</mu2>
+    <selfCollide>true</selfCollide>
+  </gazebo>
+  <gazebo reference="fl_steer_1">
+    <material>Gazebo/DarkGrey</material>
+    <mu1>0.2</mu1>
+    <mu2>0.2</mu2>
+    <selfCollide>true</selfCollide>
+  </gazebo>
+  <gazebo reference="br_steer_1">
+    <material>Gazebo/DarkGrey</material>
+    <mu1>0.2</mu1>
+    <mu2>0.2</mu2>
+    <selfCollide>true</selfCollide>
+  </gazebo>
+  <gazebo reference="bl_steer_1">
     <material>Gazebo/DarkGrey</material>
     <mu1>0.2</mu1>

File: description/urdf/autocar_joint_gazebo_control.xacro (robot description, xacro)
@@ -22,6 +22,10 @@
       <update_rate>100</update_rate>
       <!-- Name of joints in the model whose states will be published. -->
-      <joint_name>l_steer</joint_name>
-      <joint_name>r_steer</joint_name>
+      <joint_name>fl_steer</joint_name>
+      <joint_name>fr_steer</joint_name>
+      <xacro:if value="$(arg use_4ws)">
+        <joint_name>bl_steer</joint_name>
+        <joint_name>br_steer</joint_name>
+      </xacro:if>
       <joint_name>fl_axle</joint_name>
       <joint_name>fr_axle</joint_name>

File: description/urdf/autocar_ros2_control.xacro (robot description, xacro)
@@ -42,5 +42,5 @@
       <state_interface name="effort"/>
     </joint>
-    <joint name="r_steer">
+    <joint name="fr_steer">
       <command_interface name="position">
         <param name="min">-0.85</param>
@@ -51,5 +51,5 @@
       <state_interface name="effort"/>
     </joint>
-    <joint name="l_steer">
+    <joint name="fl_steer">
       <command_interface name="position">
         <param name="min">-0.85</param>
@@ -60,4 +60,24 @@
       <state_interface name="effort"/>
     </joint>
+    <xacro:if value="$(arg use_4ws)">
+      <joint name="br_steer">
+        <command_interface name="position">
+          <param name="min">-0.85</param>
+          <param name="max">0.85</param>
+        </command_interface>
+        <state_interface name="position"/>
+        <state_interface name="velocity"/>
+        <state_interface name="effort"/>
+      </joint>
+      <joint name="bl_steer">
+        <command_interface name="position">
+          <param name="min">-0.85</param>
+          <param name="max">0.85</param>
+        </command_interface>
+        <state_interface name="position"/>
+        <state_interface name="velocity"/>
+        <state_interface name="effort"/>
+      </joint>
+    </xacro:if>
   </ros2_control>
   <gazebo>

Commit message: Add p3d gazebo_control for ground-truth odom

File: description/urdf/autocar.urdf.xacro (robot description, xacro)
@@ -5,4 +5,5 @@
   <xacro:arg name="gazebo_control_config" default="autocar_ackermann_gazebo_control.xacro"/>
   <xacro:include filename="autocar_core.xacro" />
+  <xacro:include filename="autocar_p3d_gazebo_control.xacro" />
   <xacro:if value="$(arg use_ros2_control)">
     <xacro:include filename="autocar_ros2_control.xacro" />

File: description/urdf/autocar_core.xacro (robot description, xacro)
@@ -1,4 +1,5 @@
 <?xml version="1.0"?>
 <robot xmlns:xacro="http://www.ros.org/wiki/xacro">
+  <origin xyz="0 0 0" rpy="0 0 0" />
   <!-- RVIZ MATERIAL COLOUR -->
   <material name="silver">
